Commit message: random heightfield terrain

File: motion_imitation/utilities/a1/a1_tactile.urdf (robot description, URDF)
Before this commit: robot a1_description, 18 links, 17 joints
Links:
- link toeFL: geometry collision sphere radius=0.04
- link toeFR: geometry collision sphere radius=0.04
- link toeRL: geometry collision sphere radius=0.04
- link toeRR: geometry collision sphere radius=0.04
